File: cti20-to-arm20-adapter.kicad_sch (KiCad schematic)
At the start: 3 parts

Commit message: ok
Parts:
- removed J?: Conn_ARM_JTAG_SWD_20, symbol Connector:Conn_ARM_JTAG_SWD_20
- removed J?: Conn_ARM_JTAG_SWD_10, symbol Connector:Conn_ARM_JTAG_SWD_10
- added J1: Conn_02x10_Odd_Even, Connector_PinHeader_2.54mm:PinHeader_2x10_P2.54mm_Vertical_SMD, symbol Connector_Generic:Conn_02x10_Odd_Even
- J2: renamed from J?; footprint (none) -> Connector_PinSocket_1.27mm:PinSocket_2x10_P1.27mm_Vertical_SMD
Connections:
- net TMS: now reaches J2.1 (Pin_1)
- net TMS: now also J1.7 (Pin_7)
- net GND: now reaches J2.10 (Pin_10)
- net GND: now also J2.12 (Pin_12), J2.16 (Pin_16), J2.20 (Pin_20), J2.4 (Pin_4), J2.8 (Pin_8), J1.10 (Pin_10), J1.12 (Pin_12), J1.14 (Pin_14), J1.16 (Pin_16), J1.18 (Pin_18), J1.20 (Pin_20), J1.4 (Pin_4), J1.6 (Pin_6), J1.8 (Pin_8)
- net TCK: now reaches J2.11 (Pin_11)
- net TCK: now also J1.9 (Pin_9)
- net SRST_N: now reaches J2.15 (Pin_15)
- net SRST_N: now also J1.15 (Pin_15)
- net TRST_N: now reaches J2.2 (Pin_2)
- net TRST_N: now also J1.3 (Pin_3)
- net TDI: now reaches J2.3 (Pin_3)
- net TDI: now also J1.5 (Pin_5)
- net VDD: now reaches J2.5 (Pin_5)
- net VDD: now also J1.1 (Pin_1)
- net TDO: now reaches J2.7 (Pin_7)
- net TDO: now also J1.13 (Pin_13)
- net RTCK: now reaches J2.9 (Pin_9)
- net RTCK: now also J1.11 (Pin_11)
- no-connect marks 0 -> 9
Other:
- note added: "ARM 20-PIN"
- note added: "CTI-20-PIN"
- note added: "example: https://github.com/mmorawiec/BeagleBone-Black-JTAG-Adapters/blob/master/BBB_JTAG_CTI20_SMT_ARM20_SMT/BBB_JTAG_CTI20_SMT_ARM20_SMT.pdf"
- note added: "key"
- moved on the sheet: J2
